File: hardware/electrical/encoder.kicad_sch (KiCad schematic)
At the start: 9 parts

Commit message: Schematic rev. 2 Add second microcontroller to handle encoder, buttons and LEDs Remove external pull-up resistors Simplify LED driver circuits Remove debouncing capacitors Rename SPI connections with standard names Use SPI1 rather than SPI2 Isolate GNDD and GLED
Parts:
- removed C?: 47n, symbol Device:C
- removed R?: 5k2, symbol Device:R
- added D? (x6): WHITE, symbol Device:LED
- added Q?: PMBF170, symbol Device:Q_NMOS_GSD
- added R?: R, symbol Device:R
Connections:
- net GND renamed GNDD
- new net: D?.1 (K), D?.1 (K), Q?.3 (D)
- new net: D?.1 (K), D?.2 (A) (x4)
- new net: D?.2 (A), D?.2 (A), R?.2
- new net ENCODER_LED: Q?.1 (G)
- new net GLED: Q?.2 (S)
- new net VLED: R?.1
Other:
- company: (none) -> © ANDREI ANATSKA, FRANK PLOWMAN 2022
- moved on the sheet: C?, R?, SW?
